File: 42688-p-module.kicad_sch (KiCad schematic)
At the start: 12 parts, among them IC1 ICM-42688-P, J1 Conn_01x06_Pin, J2 Conn_01x01_Pin, X1 O3232768151850

Commit message: support SPI
Parts:
- added R4: 3.9k, Resistor_SMD:R_0402_1005Metric, symbol Device:R
Connections:
- net +3.3V: now also R4.1; no longer IC1.12 (AP_CS)
- net CS: now reaches J1.5 (Pin_5)
- net CS: now also IC1.12 (AP_CS), R4.2
- no-connect marks 6 -> 5
